File: embedded_project_design.kicad_sch (KiCad schematic)
At the start: 9 parts, among them J1 Conn_01x04(TO PC FAN), J2 USB_B (To PC for Serial commu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, SW1 SW_Push, U1 STM32L432KCUx

Commit message: t push origin main
Connections:
- net at J1.1 (Pin_1), U1.12 (PA6): now also U1.7 (PA1)
- new net: LCDScreen2. (VCC), U1.13 (PA7)
- new net: LCDScreen2. (VCC), RotaryEncoder. (Clk), U1.26 (PB3)
Other:
- moved on the sheet: BZ1, D1, J1, J2, R1, RotaryEncoder, SW1
